Commit message: nav

File: twowheel_drive/urdf/2w.urdf (robot description, URDF)
Before this commit: robot twowheel, 6 links, 5 joints
Links:
- removed link world_link
- added link base_footprint
Joints:
- removed joint world_to_base
- added joint base_footprint_joint: type fixed, parent base_footprint, child base_link, origin xyz=0 0 0.5 rpy=0 0 0
- joint Revolute_4: limit effort=1000 velocity=1000 -> (none)
- joint Revolute_5: limit effort=1000 velocity=1000 -> (none)
